File: subleq.sch (KiCad schematic (older format))
At the start: 8 parts, among them U1 74HC107, U10 74HC107, U2 74HC107, U3 74HC107, U4 74HC107, U5 74HC107, U6 74HC11, U7 74HC11

Commit message: started pcb file
Parts:
- U1, U2, U3, U4, U5, U6, U7: footprint (none) -> Package_DIP:DIP-14_W7.62mm
- U5: renamed from U10; footprint (none) -> Package_DIP:DIP-14_W7.62mm
Connections:
- net labels added: VCC
- net labels removed: VDD
Changed lines of the file:
@@
 EESchema Schematic File Version 4
+LIBS:subleq-cache
 EELAYER 26 0
 EELAYER END
@@
 F 0 "U1" H 4100 3417 50  0000 C CNN
 F 1 "74HC107" H 4100 3326 50  0000 C CNN
-F 2 "" H 4100 3050 50  0001 C CNN
+F 2 "Package_DIP:DIP-14_W7.62mm" H 4100 3050 50  0001 C CNN
 F 3 "http://www.ti.com/lit/gpn/sn74LS107" H 4100 3050 50  0001 C CNN
 	1    4100 3050
@@
 F 0 "U1" H 5200 3417 50  0000 C CNN
 F 1 "74HC107" H 5200 3326 50  0000 C CNN
-F 2 "" H 5200 3050 50  0001 C CNN
+F 2 "Package_DIP:DIP-14_W7.62mm" H 5200 3050 50  0001 C CNN
 F 3 "http://www.ti.com/lit/gpn/sn74LS107" H 5200 3050 50  0001 C CNN
 	2    5200 3050
@@
 F 0 "U2" H 6000 3417 50  0000 C CNN
 F 1 "74HC107" H 6000 3326 50  0000 C CNN
-F 2 "" H 6000 3050 50  0001 C CNN
+F 2 "Package_DIP:DIP-14_W7.62mm" H 6000 3050 50  0001 C CNN
 F 3 "http://www.ti.com/lit/gpn/sn74LS107" H 6000 3050 50  0001 C CNN
 	1    6000 3050
@@
 F 0 "U2" H 6800 3417 50  0000 C CNN
 F 1 "74HC107" H 6800 3326 50  0000 C CNN
-F 2 "" H 6800 3050 50  0001 C CNN
+F 2 "Package_DIP:DIP-14_W7.62mm" H 6800 3050 50  0001 C CNN
 F 3 "http://www.ti.com/lit/gpn/sn74LS107" H 6800 3050 50  0001 C CNN
 	2    6800 3050
@@
 F 0 "U3" H 7600 3417 50  0000 C CNN
 F 1 "74HC107" H 7600 3326 50  0000 C CNN
-F 2 "" H 7600 3050 50  0001 C CNN
+F 2 "Package_DIP:DIP-14_W7.62mm" H 7600 3050 50  0001 C CNN
 F 3 "http://www.ti.com/lit/gpn/sn74LS107" H 7600 3050 50  0001 C CNN
 	1    7600 3050
@@
 F 0 "U3" H 8400 3417 50  0000 C CNN
 F 1 "74HC107" H 8400 3326 50  0000 C CNN
-F 2 "" H 8400 3050 50  0001 C CNN
+F 2 "Package_DIP:DIP-14_W7.62mm" H 8400 3050 50  0001 C CNN
 F 3 "http://www.ti.com/lit/gpn/sn74LS107" H 8400 3050 50  0001 C CNN
 	2    8400 3050
@@
 F 0 "U4" H 9200 3417 50  0000 C CNN
 F 1 "74HC107" H 9200 3326 50  0000 C CNN
-F 2 "" H 9200 3050 50  0001 C CNN
+F 2 "Package_DIP:DIP-14_W7.62mm" H 9200 3050 50  0001 C CNN
 F 3 "http://www.ti.com/lit/gpn/sn74LS107" H 9200 3050 50  0001 C CNN
 	1    9200 3050
@@
 F 0 "U4" H 10000 3417 50  0000 C CNN
 F 1 "74HC107" H 10000 3326 50  0000 C CNN
-F 2 "" H 10000 3050 50  0001 C CNN
+F 2 "Package_DIP:DIP-14_W7.62mm" H 10000 3050 50  0001 C CNN
 F 3 "http://www.ti.com/lit/gpn/sn74LS107" H 10000 3050 50  0001 C CNN
 	2    10000 3050
@@
 F 0 "U5" H 10800 3417 50  0000 C CNN
 F 1 "74HC107" H 10800 3326 50  0000 C CNN
-F 2 "" H 10800 3050 50  0001 C CNN
+F 2 "Package_DIP:DIP-14_W7.62mm" H 10800 3050 50  0001 C CNN
 F 3 "http://www.ti.com/lit/gpn/sn74LS107" H 10800 3050 50  0001 C CNN
 	1    10800 3050
@@
 $EndComp
 $Comp
-L 74xx:74LS107 U10
-U 1 1 5C4CCA35
+L 74xx:74LS107 U5
+U 2 1 5C4CCA35
 P 11600 3050
-F 0 "U10" H 11600 3417 50  0000 C CNN
+F 0 "U5" H 11600 3417 50  0000 C CNN
 F 1 "74HC107" H 11600 3326 50  0000 C CNN
-F 2 "" H 11600 3050 50  0001 C CNN
+F 2 "Package_DIP:DIP-14_W7.62mm" H 11600 3050 50  0001 C CNN
 F 3 "http://www.ti.com/lit/gpn/sn74LS107" H 11600 3050 50  0001 C CNN
-	1    11600 3050
+	2    11600 3050
 	1    0    0    -1
 $EndComp
@@
 F 0 "U6" H 12550 5125 50  0000 C CNN
 F 1 "74HC11" H 12550 5034 50  0000 C CNN
-F 2 "" H 12550 4800 50  0001 C CNN
+F 2 "Package_DIP:DIP-14_W7.62mm" H 12550 4800 50  0001 C CNN
 F 3 "http://www.ti.com/lit/gpn/sn74LS11" H 12550 4800 50  0001 C CNN
 	1    12550 4800
@@
 F 0 "U6" H 12550 5675 50  0000 C CNN
 F 1 "74HC11" H 12550 5584 50  0000 C CNN
-F 2 "" H 12550 5350 50  0001 C CNN
+F 2 "Package_DIP:DIP-14_W7.62mm" H 12550 5350 50  0001 C CNN
 F 3 "http://www.ti.com/lit/gpn/sn74LS11" H 12550 5350 50  0001 C CNN
 	2    12550 5350
@@
 F 0 "U6" H 12550 6225 50  0000 C CNN
 F 1 "74HC11" H 12550 6134 50  0000 C CNN
-F 2 "" H 12550 5900 50  0001 C CNN
+F 2 "Package_DIP:DIP-14_W7.62mm" H 12550 5900 50  0001 C CNN
 F 3 "http://www.ti.com/lit/gpn/sn74LS11" H 12550 5900 50  0001 C CNN
 	3    12550 5900
@@
 F 0 "U7" H 12550 6775 50  0000 C CNN
 F 1 "74HC11" H 12550 6684 50  0000 C CNN
-F 2 "" H 12550 6450 50  0001 C CNN
+F 2 "Package_DIP:DIP-14_W7.62mm" H 12550 6450 50  0001 C CNN
 F 3 "http://www.ti.com/lit/gpn/sn74LS11" H 12550 6450 50  0001 C CNN
 	1    12550 6450
@@
 F 0 "U7" H 12550 7325 50  0000 C CNN
 F 1 "74HC11" H 12550 7234 50  0000 C CNN
-F 2 "" H 12550 7000 50  0001 C CNN
+F 2 "Package_DIP:DIP-14_W7.62mm" H 12550 7000 50  0001 C CNN
 F 3 "http://www.ti.com/lit/gpn/sn74LS11" H 12550 7000 50  0001 C CNN
 	2    12550 7000
@@
 F 0 "U7" H 13400 7025 50  0000 C CNN
 F 1 "74HC11" H 13400 6934 50  0000 C CNN
-F 2 "" H 13400 6700 50  0001 C CNN
+F 2 "Package_DIP:DIP-14_W7.62mm" H 13400 6700 50  0001 C CNN
 F 3 "http://www.ti.com/lit/gpn/sn74LS11" H 13400 6700 50  0001 C CNN
 	3    13400 6700
@@
 Wire Wire Line
 	13050 6600 13050 6350
-$Comp
-L power:VDD #PWR01
-U 1 1 5C60E2A3
-P 13050 6350
-F 0 "#PWR01" H 13050 6200 50  0001 C CNN
-F 1 "VDD" H 13067 6523 50  0000 C CNN
-F 2 "" H 13050 6350 50  0001 C CNN
-F 3 "" H 13050 6350 50  0001 C CNN
-	1    13050 6350
-	1    0    0    -1
-$EndComp
 Wire Wire Line
 	13700 6700 13800 6700
@@
 Connection ~ 6350 3150
 Connection ~ 5550 3150
+$Comp
+L power:VCC #PWR?
+U 1 1 5C4E2EE5
+P 13050 6350
+F 0 "#PWR?" H 13050 6200 50  0001 C CNN
+F 1 "VCC" H 13067 6523 50  0000 C CNN
+F 2 "" H 13050 6350 50  0001 C CNN
+F 3 "" H 13050 6350 50  0001 C CNN
+	1    13050 6350
+	1    0    0    -1
+$EndComp
 $EndSCHEMATC
