File: subleq.sch (KiCad schematic (older format))
At the start: 0 parts

Commit message: backup before registers alu split
Changed lines of the file:
@@
 $Descr USLedger 17000 11000
 encoding utf-8
-Sheet 1 4
+Sheet 1 6
 Title ""
 Date ""
@@
 $EndSheet
 $Sheet
-S 12300 6200 900  700
-U 5C4D6ED1
+S 12300 6200 950  700
+U 5CB820A3
+F0 "REGISTERS_AND_ALU" 50
+F1 "registers_and_alu.sch" 50
+$EndSheet
+$Sheet
+S 13450 6200 1000 700
+U 5CBABD04
+F0 "MEMORY" 50
+F1 "memory.sch" 50
+$EndSheet
+$Sheet
+S 14650 6200 1050 700
+U 5CBC693B
 F0 "REGISTERS" 50
 F1 "registers.sch" 50
