File: program_counter.sch (KiCad schematic (older format))
At the start: 5 parts, among them U10 74HC161, U11 74HC161, U12 74HC161, U8 74HC04, U9 74HC161

Commit message: backup before registers alu split
Connections:
- net PC_D0: no longer names the net of U9.3 (D0)
- net PC_D1: no longer names the net of U9.4 (D1)
- net PC_D10: no longer names the net of U11.5 (D2)
- net PC_D11: no longer names the net of U11.6 (D3)
- net PC_D12: no longer names the net of U12.3 (D0)
- net PC_D13: no longer names the net of U12.4 (D1)
- net PC_D14: no longer names the net of U12.5 (D2)
- net PC_D15: no longer names the net of U12.6 (D3)
- net PC_D2: no longer names the net of U9.5 (D2)
- net PC_D3: no longer names the net of U9.6 (D3)
- net PC_D4: no longer names the net of U10.3 (D0)
- net PC_D5: no longer names the net of U10.4 (D1)
- net PC_D6: no longer names the net of U10.5 (D2)
- net PC_D7: no longer names the net of U10.6 (D3)
- net PC_D8: no longer names the net of U11.3 (D0)
- net PC_D9: no longer names the net of U11.4 (D1)
Changed lines of the file:
@@
 $Descr USLedger 17000 11000
 encoding utf-8
-Sheet 3 4
+Sheet 3 6
 Title ""
 Date ""
@@
 PC_Q
 Text GLabel 6850 3200 0    50   Input ~ 0
-PC_D
+MAR_Q
 Wire Wire Line
 	8150 4100 7850 4100
@@
 Wire Wire Line
 	7150 3600 8150 3600
-Text Label 7250 3500 0    50   ~ 0
-PC_D0
-Text Label 7250 3600 0    50   ~ 0
-PC_D1
-Text Label 7250 3700 0    50   ~ 0
-PC_D2
-Text Label 7250 3800 0    50   ~ 0
-PC_D3
-Text Label 7250 4950 0    50   ~ 0
-PC_D4
-Text Label 7250 5050 0    50   ~ 0
-PC_D5
-Text Label 7250 5150 0    50   ~ 0
-PC_D6
-Text Label 7250 5250 0    50   ~ 0
-PC_D7
-Text Label 7250 6400 0    50   ~ 0
-PC_D8
-Text Label 7250 6500 0    50   ~ 0
-PC_D9
-Text Label 7250 6600 0    50   ~ 0
-PC_D10
-Text Label 7250 6700 0    50   ~ 0
-PC_D11
-Text Label 7250 7850 0    50   ~ 0
-PC_D12
-Text Label 7250 7950 0    50   ~ 0
-PC_D13
-Text Label 7250 8050 0    50   ~ 0
-PC_D14
-Text Label 7250 8150 0    50   ~ 0
-PC_D15
 Text Label 9550 3500 2    50   ~ 0
 PC_Q0

Commit message: done for the night passing drc
Connections:
- net MAR_Q0: now reaches U9.3 (D0)
- net MAR_Q1: now reaches U9.4 (D1)
- net MAR_Q2: now reaches U9.5 (D2)
- net MAR_Q3: now reaches U9.6 (D3)
- net MAR_Q4: now reaches U10.3 (D0)
- net MAR_Q5: now reaches U10.4 (D1)
- net MAR_Q6: now reaches U10.5 (D2)
- net MAR_Q7: now reaches U10.6 (D3)
- net MAR_Q8: now reaches U11.3 (D0)
- net MAR_Q9: now reaches U11.4 (D1)
- net MAR_Q10: now reaches U11.5 (D2)
- net MAR_Q11: now reaches U11.6 (D3)
- net MAR_Q12: now reaches U12.3 (D0)
- net MAR_Q13: now reaches U12.4 (D1)
- net MAR_Q14: now reaches U12.5 (D2)
- net MAR_Q15: now reaches U12.6 (D3)
- net ~PC_INC renamed ~INC_PC
Changed lines of the file:
@@
 $Descr USLedger 17000 11000
 encoding utf-8
-Sheet 3 6
+Sheet 3 7
 Title ""
 Date ""
@@
 	9700 3200 9900 3200
 Text GLabel 9900 3200 2    50   Output ~ 0
-PC_Q
+PC_Q[0..15]
 Text GLabel 6850 3200 0    50   Input ~ 0
-MAR_Q
+MAR_Q[0..15]
 Wire Wire Line
 	8150 4100 7850 4100
@@
 	7150 2450 6850 2450
 Text GLabel 6850 2450 0    50   Input ~ 0
-~PC_INC
+~INC_PC
 Wire Wire Line
 	7150 3600 8150 3600
@@
 Wire Bus Line
 	9700 3200 9700 8050
+Text Label 7250 3500 0    50   ~ 0
+MAR_Q0
+Text Label 7250 3600 0    50   ~ 0
+MAR_Q1
+Text Label 7250 3700 0    50   ~ 0
+MAR_Q2
+Text Label 7250 3800 0    50   ~ 0
+MAR_Q3
+Text Label 7250 4950 0    50   ~ 0
+MAR_Q4
+Text Label 7250 5050 0    50   ~ 0
+MAR_Q5
+Text Label 7250 5150 0    50   ~ 0
+MAR_Q6
+Text Label 7250 5250 0    50   ~ 0
+MAR_Q7
+Text Label 7250 6400 0    50   ~ 0
+MAR_Q8
+Text Label 7250 6500 0    50   ~ 0
+MAR_Q9
+Text Label 7250 6600 0    50   ~ 0
+MAR_Q10
+Text Label 7250 6700 0    50   ~ 0
+MAR_Q11
+Text Label 7250 7850 0    50   ~ 0
+MAR_Q12
+Text Label 7250 7950 0    50   ~ 0
+MAR_Q13
+Text Label 7250 8050 0    50   ~ 0
+MAR_Q14
+Text Label 7250 8150 0    50   ~ 0
+MAR_Q15
 $EndSCHEMATC
