File: alu.sch (KiCad schematic (older format))
At the start: 15 parts

Commit message: done for the night passing drc
Parts:
- gave numbers to parts that had none: 8
Connections:
- net ~MEM_WR renamed ~WR_MEM
Changed lines of the file:
@@
 $Descr USLedger 17000 11000
 encoding utf-8
-Sheet 6 6
+Sheet 6 7
 Title ""
 Date ""
@@
 AR Path="/5C4D6ED1/5C4E2FE6" Ref="U?"  Part="1"
 AR Path="/5CB820A3/5C4E2FE6" Ref="U?"  Part="1"
-AR Path="/5C4D52FD/5C4E2FE6" Ref="U?"  Part="1"
-F 0 "U?" H 8350 5300 50  0000 C CNN
+AR Path="/5C4D52FD/5C4E2FE6" Ref="U24"  Part="1"
+F 0 "U24" H 8350 5300 50  0000 C CNN
 F 1 "74HC283" H 8600 4000 50  0000 C CNN
 F 2 "" H 8600 4650 50  0001 C CNN
@@
 AR Path="/5C4D6ED1/5C4E2FED" Ref="U?"  Part="1"
 AR Path="/5CB820A3/5C4E2FED" Ref="U?"  Part="1"
-AR Path="/5C4D52FD/5C4E2FED" Ref="U?"  Part="1"
-F 0 "U?" H 8350 6800 50  0000 C CNN
+AR Path="/5C4D52FD/5C4E2FED" Ref="U25"  Part="1"
+F 0 "U25" H 8350 6800 50  0000 C CNN
 F 1 "74HC283" H 8600 5500 50  0000 C CNN
 F 2 "" H 8600 6150 50  0001 C CNN
@@
 AR Path="/5C4D6ED1/5C4E2FFB" Ref="U?"  Part="2"
 AR Path="/5CB820A3/5C4E2FFB" Ref="U?"  Part="2"
-AR Path="/5C4D52FD/5C4E2FFB" Ref="U?"  Part="2"
-F 0 "U?" H 5700 2300 50  0000 C CNN
+AR Path="/5C4D52FD/5C4E2FFB" Ref="U8"  Part="2"
+F 0 "U8" H 5700 2300 50  0000 C CNN
 F 1 "74HC04" H 5700 1850 50  0000 C CNN
 F 2 "Package_DIP:DIP-14_W7.62mm" H 5700 2100 50  0001 C CNN
@@
 AR Path="/5C4D6ED1/5C4E3002" Ref="U?"  Part="4"
 AR Path="/5CB820A3/5C4E3002" Ref="U?"  Part="4"
-AR Path="/5C4D52FD/5C4E3002" Ref="U?"  Part="4"
-F 0 "U?" H 5700 2950 50  0000 C CNN
+AR Path="/5C4D52FD/5C4E3002" Ref="U22"  Part="4"
+F 0 "U22" H 5700 2950 50  0000 C CNN
 F 1 "74HC04" H 5700 2500 50  0000 C CNN
 F 2 "Package_DIP:DIP-14_W7.62mm" H 5700 2750 50  0001 C CNN
@@
 AR Path="/5C4D6ED1/5C4E3009" Ref="U?"  Part="6"
 AR Path="/5CB820A3/5C4E3009" Ref="U?"  Part="6"
-AR Path="/5C4D52FD/5C4E3009" Ref="U?"  Part="6"
-F 0 "U?" H 5700 3600 50  0000 C CNN
+AR Path="/5C4D52FD/5C4E3009" Ref="U8"  Part="6"
+F 0 "U8" H 5700 3600 50  0000 C CNN
 F 1 "74HC04" H 5700 3150 50  0000 C CNN
 F 2 "Package_DIP:DIP-14_W7.62mm" H 5700 3400 50  0001 C CNN
@@
 AR Path="/5C4D6ED1/5C4E3010" Ref="U?"  Part="2"
 AR Path="/5CB820A3/5C4E3010" Ref="U?"  Part="2"
-AR Path="/5C4D52FD/5C4E3010" Ref="U?"  Part="2"
-F 0 "U?" H 5700 4250 50  0000 C CNN
+AR Path="/5C4D52FD/5C4E3010" Ref="U22"  Part="2"
+F 0 "U22" H 5700 4250 50  0000 C CNN
 F 1 "74HC04" H 5700 3800 50  0000 C CNN
 F 2 "Package_DIP:DIP-14_W7.62mm" H 5700 4050 50  0001 C CNN
@@
 AR Path="/5C4D6ED1/5C4E3017" Ref="U?"  Part="1"
 AR Path="/5CB820A3/5C4E3017" Ref="U?"  Part="1"
-AR Path="/5C4D52FD/5C4E3017" Ref="U?"  Part="1"
-F 0 "U?" H 6350 2000 50  0000 C CNN
+AR Path="/5C4D52FD/5C4E3017" Ref="U22"  Part="1"
+F 0 "U22" H 6350 2000 50  0000 C CNN
 F 1 "74HC04" H 6350 1550 50  0000 C CNN
 F 2 "Package_DIP:DIP-14_W7.62mm" H 6350 1800 50  0001 C CNN
@@
 AR Path="/5C4D6ED1/5C4E301E" Ref="U?"  Part="3"
 AR Path="/5CB820A3/5C4E301E" Ref="U?"  Part="3"
-AR Path="/5C4D52FD/5C4E301E" Ref="U?"  Part="3"
-F 0 "U?" H 6350 2650 50  0000 C CNN
+AR Path="/5C4D52FD/5C4E301E" Ref="U8"  Part="3"
+F 0 "U8" H 6350 2650 50  0000 C CNN
 F 1 "74HC04" H 6350 2200 50  0000 C CNN
 F 2 "Package_DIP:DIP-14_W7.62mm" H 6350 2450 50  0001 C CNN
@@
 AR Path="/5C4D6ED1/5C4E3025" Ref="U?"  Part="5"
 AR Path="/5CB820A3/5C4E3025" Ref="U?"  Part="5"
-AR Path="/5C4D52FD/5C4E3025" Ref="U?"  Part="5"
-F 0 "U?" H 6350 3300 50  0000 C CNN
+AR Path="/5C4D52FD/5C4E3025" Ref="U8"  Part="5"
+F 0 "U8" H 6350 3300 50  0000 C CNN
 F 1 "74HC04" H 6350 2850 50  0000 C CNN
 F 2 "Package_DIP:DIP-14_W7.62mm" H 6350 3100 50  0001 C CNN
@@
 AR Path="/5C4D6ED1/5C4E302C" Ref="U?"  Part="1"
 AR Path="/5CB820A3/5C4E302C" Ref="U?"  Part="1"
-AR Path="/5C4D52FD/5C4E302C" Ref="U?"  Part="1"
-F 0 "U?" H 6350 3950 50  0000 C CNN
+AR Path="/5C4D52FD/5C4E302C" Ref="U23"  Part="1"
+F 0 "U23" H 6350 3950 50  0000 C CNN
 F 1 "74HC04" H 6350 3500 50  0000 C CNN
 F 2 "Package_DIP:DIP-14_W7.62mm" H 6350 3750 50  0001 C CNN
@@
 AR Path="/5C4D6ED1/5C4E306F" Ref="#PWR?"  Part="1"
 AR Path="/5CB820A3/5C4E306F" Ref="#PWR?"  Part="1"
-AR Path="/5C4D52FD/5C4E306F" Ref="#PWR?"  Part="1"
-F 0 "#PWR?" H 8000 3750 50  0001 C CNN
+AR Path="/5C4D52FD/5C4E306F" Ref="#PWR06"  Part="1"
+F 0 "#PWR06" H 8000 3750 50  0001 C CNN
 F 1 "VCC" H 8017 4073 50  0000 C CNN
 F 2 "" H 8000 3900 50  0001 C CNN
@@
 AR Path="/5C4D6ED1/5C4E3078" Ref="U?"  Part="3"
 AR Path="/5CB820A3/5C4E3078" Ref="U?"  Part="3"
-AR Path="/5C4D52FD/5C4E3078" Ref="U?"  Part="3"
-F 0 "U?" H 10850 6650 50  0000 C CNN
+AR Path="/5C4D52FD/5C4E3078" Ref="U22"  Part="3"
+F 0 "U22" H 10850 6650 50  0000 C CNN
 F 1 "74HC04" H 10850 6200 50  0000 C CNN
 F 2 "Package_DIP:DIP-14_W7.62mm" H 10850 6450 50  0001 C CNN
@@
 AR Path="/5C4D6ED1/5C4E3080" Ref="U?"  Part="1"
 AR Path="/5CB820A3/5C4E3080" Ref="U?"  Part="1"
-AR Path="/5C4D52FD/5C4E3080" Ref="U?"  Part="1"
-F 0 "U?" H 10700 8950 50  0000 L CNN
+AR Path="/5C4D52FD/5C4E3080" Ref="U26"  Part="1"
+F 0 "U26" H 10700 8950 50  0000 L CNN
 F 1 "74HC688" H 10850 6850 50  0000 L CNN
 F 2 "" H 11000 7900 50  0001 C CNN
@@
 AR Path="/5C4D6ED1/5C4E30A1" Ref="#PWR?"  Part="1"
 AR Path="/5CB820A3/5C4E30A1" Ref="#PWR?"  Part="1"
-AR Path="/5C4D52FD/5C4E30A1" Ref="#PWR?"  Part="1"
-F 0 "#PWR?" H 10400 8750 50  0001 C CNN
+AR Path="/5C4D52FD/5C4E30A1" Ref="#PWR07"  Part="1"
+F 0 "#PWR07" H 10400 8750 50  0001 C CNN
 F 1 "GND" H 10405 8827 50  0000 C CNN
 F 2 "" H 10400 9000 50  0001 C CNN
@@
 AR Path="/5C4D6ED1/5C4E30B7" Ref="U?"  Part="1"
 AR Path="/5CB820A3/5C4E30B7" Ref="U?"  Part="1"
-AR Path="/5C4D52FD/5C4E30B7" Ref="U?"  Part="1"
-F 0 "U?" H 12000 7225 50  0000 C CNN
+AR Path="/5C4D52FD/5C4E30B7" Ref="U27"  Part="1"
+F 0 "U27" H 12000 7225 50  0000 C CNN
 F 1 "74HC32" H 12000 7134 50  0000 C CNN
 F 2 "" H 12000 6900 50  0001 C CNN
@@
 AR Path="/5C4D6ED1/5C4E30C2" Ref="U?"  Part="2"
 AR Path="/5CB820A3/5C4E30C2" Ref="U?"  Part="2"
-AR Path="/5C4D52FD/5C4E30C2" Ref="U?"  Part="2"
-F 0 "U?" H 12800 7325 50  0000 C CNN
+AR Path="/5C4D52FD/5C4E30C2" Ref="U27"  Part="2"
+F 0 "U27" H 12800 7325 50  0000 C CNN
 F 1 "74HC32" H 12800 7234 50  0000 C CNN
 F 2 "" H 12800 7000 50  0001 C CNN
@@
 ~LD_PC
 Text GLabel 11400 3500 0    50   Input ~ 0
-~MEM_WR
+~WR_MEM
 Wire Bus Line
 	13450 3850 13650 3850
 Text GLabel 13650 3850 2    50   Output ~ 0
-MEM_DQ
+MEM_DQ[0..7]
 Wire Wire Line
 	9100 4150 10300 4150
@@
 AR Path="/5C4D6ED1/5C4E30DA" Ref="U?"  Part="1"
 AR Path="/5CB820A3/5C4E30DA" Ref="U?"  Part="1"
-AR Path="/5C4D52FD/5C4E30DA" Ref="U?"  Part="1"
-F 0 "U?" H 12200 5417 50  0000 C CNN
+AR Path="/5C4D52FD/5C4E30DA" Ref="U28"  Part="1"
+F 0 "U28" H 12200 5417 50  0000 C CNN
 F 1 "74HC541" H 12200 5326 50  0000 C CNN
 F 2 "" H 12200 4650 50  0001 C CNN
@@
 	4350 3050 4350 3950
 Text GLabel 4150 3050 0    50   Input ~ 0
-A
+A[0..7]
 Text GLabel 4150 4550 0    50   Input ~ 0
-B
+B[0..7]
 Text Label 4550 3350 0    50   ~ 0
 A0

Commit message: calling it a night
Parts:
- U24, U25: footprint (none) -> Package_DIP:DIP-16_W7.62mm
- U26, U28: footprint (none) -> Package_DIP:DIP-20_W7.62mm
- U27: footprint (none) -> Package_DIP:DIP-14_W7.62mm
Changed lines of the file:
@@
 F 0 "U24" H 8350 5300 50  0000 C CNN
 F 1 "74HC283" H 8600 4000 50  0000 C CNN
-F 2 "" H 8600 4650 50  0001 C CNN
+F 2 "Package_DIP:DIP-16_W7.62mm" H 8600 4650 50  0001 C CNN
 F 3 "http://www.ti.com/lit/gpn/sn74LS283" H 8600 4650 50  0001 C CNN
 	1    8600 4650
@@
 F 0 "U25" H 8350 6800 50  0000 C CNN
 F 1 "74HC283" H 8600 5500 50  0000 C CNN
-F 2 "" H 8600 6150 50  0001 C CNN
+F 2 "Package_DIP:DIP-16_W7.62mm" H 8600 6150 50  0001 C CNN
 F 3 "http://www.ti.com/lit/gpn/sn74LS283" H 8600 6150 50  0001 C CNN
 	1    8600 6150
@@
 F 0 "U26" H 10700 8950 50  0000 L CNN
 F 1 "74HC688" H 10850 6850 50  0000 L CNN
-F 2 "" H 11000 7900 50  0001 C CNN
+F 2 "Package_DIP:DIP-20_W7.62mm" H 11000 7900 50  0001 C CNN
 F 3 "http://www.ti.com/lit/gpn/sn74LS688" H 11000 7900 50  0001 C CNN
 	1    11000 7900
@@
 F 0 "U27" H 12000 7225 50  0000 C CNN
 F 1 "74HC32" H 12000 7134 50  0000 C CNN
-F 2 "" H 12000 6900 50  0001 C CNN
+F 2 "Package_DIP:DIP-14_W7.62mm" H 12000 6900 50  0001 C CNN
 F 3 "http://www.ti.com/lit/gpn/sn74LS32" H 12000 6900 50  0001 C CNN
 	1    12000 6900
@@
 F 0 "U27" H 12800 7325 50  0000 C CNN
 F 1 "74HC32" H 12800 7234 50  0000 C CNN
-F 2 "" H 12800 7000 50  0001 C CNN
+F 2 "Package_DIP:DIP-14_W7.62mm" H 12800 7000 50  0001 C CNN
 F 3 "http://www.ti.com/lit/gpn/sn74LS32" H 12800 7000 50  0001 C CNN
 	2    12800 7000
@@
 F 0 "U28" H 12200 5417 50  0000 C CNN
 F 1 "74HC541" H 12200 5326 50  0000 C CNN
-F 2 "" H 12200 4650 50  0001 C CNN
+F 2 "Package_DIP:DIP-20_W7.62mm" H 12200 4650 50  0001 C CNN
 F 3 "http://www.ti.com/lit/gpn/sn74LS541" H 12200 4650 50  0001 C CNN
 	1    12200 4650
