File: control.sch (KiCad schematic (older format))
At the start: 12 parts, among them U6 74HC11, U7 74HC11

Commit message: done for the night passing drc
Parts:
- gave numbers to parts that had none: 5
Connections:
- net ~ADDR_SEL renamed ~SEL_ADDR_PC_MAR
- net ~CLK renamed CLK
- net ~PC_INC renamed ~INC_PC
Changed lines of the file:
@@
 $Descr USLedger 17000 11000
 encoding utf-8
-Sheet 2 6
+Sheet 2 7
 Title ""
 Date ""
@@
 ~RST
 Text GLabel 3150 4050 0    50   Input ~ 0
-~CLK
+CLK
 Connection ~ 11750 3600
 Wire Wire Line
@@
 	12650 6350 13600 6350
 Text GLabel 13600 6350 2    50   Output ~ 0
-~ADDR_SEL
+~SEL_ADDR_PC_MAR
 $Comp
 L 74xx:74LS11 U?
@@
 	13500 7150 13600 7150
 Text GLabel 13600 7150 2    50   Output ~ 0
-~PC_INC
+~INC_PC
 Connection ~ 9350 4650
 Connection ~ 8550 4500
@@
 P 12850 6800
 AR Path="/5C4E9D9E" Ref="#PWR?"  Part="1"
-AR Path="/5C4E38C4/5C4E9D9E" Ref="#PWR01"  Part="1"
-F 0 "#PWR01" H 12850 6650 50  0001 C CNN
+AR Path="/5C4E38C4/5C4E9D9E" Ref="#PWR03"  Part="1"
+F 0 "#PWR03" H 12850 6650 50  0001 C CNN
 F 1 "VCC" H 12867 6973 50  0000 C CNN
 F 2 "" H 12850 6800 50  0001 C CNN
@@
 NOTE: !!! 74HC107 IS NEGATIVE EDGE TRIGGERED !!!
 $Comp
-L 74xx_modified:74HC107 U?
+L 74xx_modified:74HC107 U1
 U 1 1 5C685FFC
 P 3900 3500
-F 0 "U?" H 3900 3867 50  0000 C CNN
+F 0 "U1" H 3900 3867 50  0000 C CNN
 F 1 "74HC107" H 3900 3776 50  0000 C CNN
 F 2 "" H 3900 3500 50  0001 C CNN
@@
 $EndComp
 $Comp
-L 74xx_modified:74HC107 U?
+L 74xx_modified:74HC107 U1
 U 2 1 5C6861B7
 P 5000 3500
-F 0 "U?" H 5000 3867 50  0000 C CNN
+F 0 "U1" H 5000 3867 50  0000 C CNN
 F 1 "74HC107" H 5000 3776 50  0000 C CNN
 F 2 "" H 5000 3500 50  0001 C CNN
@@
 $EndComp
 $Comp
-L 74xx_modified:74HC107 U?
+L 74xx_modified:74HC107 U2
 U 1 1 5C690178
 P 5800 3500
-F 0 "U?" H 5800 3867 50  0000 C CNN
+F 0 "U2" H 5800 3867 50  0000 C CNN
 F 1 "74HC107" H 5800 3776 50  0000 C CNN
 F 2 "" H 5800 3500 50  0001 C CNN
@@
 $EndComp
 $Comp
-L 74xx_modified:74HC107 U?
+L 74xx_modified:74HC107 U3
 U 1 1 5C6901CC
 P 7400 3500
-F 0 "U?" H 7400 3867 50  0000 C CNN
+F 0 "U3" H 7400 3867 50  0000 C CNN
 F 1 "74HC107" H 7400 3776 50  0000 C CNN
 F 2 "" H 7400 3500 50  0001 C CNN
@@
 $EndComp
 $Comp
-L 74xx_modified:74HC107 U?
+L 74xx_modified:74HC107 U4
 U 1 1 5C690214
 P 9000 3500
-F 0 "U?" H 9000 3867 50  0000 C CNN
+F 0 "U4" H 9000 3867 50  0000 C CNN
 F 1 "74HC107" H 9000 3776 50  0000 C CNN
 F 2 "" H 9000 3500 50  0001 C CNN
@@
 $EndComp
 $Comp
-L 74xx_modified:74HC107 U?
+L 74xx_modified:74HC107 U5
 U 1 1 5C690356
 P 10600 3500
-F 0 "U?" H 10600 3867 50  0000 C CNN
+F 0 "U5" H 10600 3867 50  0000 C CNN
 F 1 "74HC107" H 10600 3776 50  0000 C CNN
 F 2 "" H 10600 3500 50  0001 C CNN
@@
 $EndComp
 $Comp
-L 74xx_modified:74HC107 U?
+L 74xx_modified:74HC107 U2
 U 2 1 5C6903F8
 P 6600 3500
-F 0 "U?" H 6600 3867 50  0000 C CNN
+F 0 "U2" H 6600 3867 50  0000 C CNN
 F 1 "74HC107" H 6600 3776 50  0000 C CNN
 F 2 "" H 6600 3500 50  0001 C CNN
@@
 $EndComp
 $Comp
-L 74xx_modified:74HC107 U?
+L 74xx_modified:74HC107 U3
 U 2 1 5C690444
 P 8200 3500
-F 0 "U?" H 8200 3867 50  0000 C CNN
+F 0 "U3" H 8200 3867 50  0000 C CNN
 F 1 "74HC107" H 8200 3776 50  0000 C CNN
 F 2 "" H 8200 3500 50  0001 C CNN
@@
 $EndComp
 $Comp
-L 74xx_modified:74HC107 U?
+L 74xx_modified:74HC107 U4
 U 2 1 5C690488
 P 9800 3500
-F 0 "U?" H 9800 3867 50  0000 C CNN
+F 0 "U4" H 9800 3867 50  0000 C CNN
 F 1 "74HC107" H 9800 3776 50  0000 C CNN
 F 2 "" H 9800 3500 50  0001 C CNN
@@
 $EndComp
 $Comp
-L 74xx_modified:74HC107 U?
+L 74xx_modified:74HC107 U5
 U 2 1 5C6905AE
 P 11400 3500
-F 0 "U?" H 11400 3867 50  0000 C CNN
+F 0 "U5" H 11400 3867 50  0000 C CNN
 F 1 "74HC107" H 11400 3776 50  0000 C CNN
 F 2 "" H 11400 3500 50  0001 C CNN

Commit message: calling it a night
Parts:
- U1, U2, U3, U4, U5: footprint (none) -> Package_DIP:DIP-14_W7.62mm
Changed lines of the file:
@@
 F 0 "U1" H 3900 3867 50  0000 C CNN
 F 1 "74HC107" H 3900 3776 50  0000 C CNN
-F 2 "" H 3900 3500 50  0001 C CNN
+F 2 "Package_DIP:DIP-14_W7.62mm" H 3900 3500 50  0001 C CNN
 F 3 "http://www.ti.com/lit/gpn/sn74LS107" H 3900 3500 50  0001 C CNN
 	1    3900 3500
@@
 F 0 "U1" H 5000 3867 50  0000 C CNN
 F 1 "74HC107" H 5000 3776 50  0000 C CNN
-F 2 "" H 5000 3500 50  0001 C CNN
+F 2 "Package_DIP:DIP-14_W7.62mm" H 5000 3500 50  0001 C CNN
 F 3 "http://www.ti.com/lit/gpn/sn74LS107" H 5000 3500 50  0001 C CNN
 	2    5000 3500
@@
 F 0 "U2" H 5800 3867 50  0000 C CNN
 F 1 "74HC107" H 5800 3776 50  0000 C CNN
-F 2 "" H 5800 3500 50  0001 C CNN
+F 2 "Package_DIP:DIP-14_W7.62mm" H 5800 3500 50  0001 C CNN
 F 3 "http://www.ti.com/lit/gpn/sn74LS107" H 5800 3500 50  0001 C CNN
 	1    5800 3500
@@
 F 0 "U3" H 7400 3867 50  0000 C CNN
 F 1 "74HC107" H 7400 3776 50  0000 C CNN
-F 2 "" H 7400 3500 50  0001 C CNN
+F 2 "Package_DIP:DIP-14_W7.62mm" H 7400 3500 50  0001 C CNN
 F 3 "http://www.ti.com/lit/gpn/sn74LS107" H 7400 3500 50  0001 C CNN
 	1    7400 3500
@@
 F 0 "U4" H 9000 3867 50  0000 C CNN
 F 1 "74HC107" H 9000 3776 50  0000 C CNN
-F 2 "" H 9000 3500 50  0001 C CNN
+F 2 "Package_DIP:DIP-14_W7.62mm" H 9000 3500 50  0001 C CNN
 F 3 "http://www.ti.com/lit/gpn/sn74LS107" H 9000 3500 50  0001 C CNN
 	1    9000 3500
@@
 F 0 "U5" H 10600 3867 50  0000 C CNN
 F 1 "74HC107" H 10600 3776 50  0000 C CNN
-F 2 "" H 10600 3500 50  0001 C CNN
+F 2 "Package_DIP:DIP-14_W7.62mm" H 10600 3500 50  0001 C CNN
 F 3 "http://www.ti.com/lit/gpn/sn74LS107" H 10600 3500 50  0001 C CNN
 	1    10600 3500
@@
 F 0 "U2" H 6600 3867 50  0000 C CNN
 F 1 "74HC107" H 6600 3776 50  0000 C CNN
-F 2 "" H 6600 3500 50  0001 C CNN
+F 2 "Package_DIP:DIP-14_W7.62mm" H 6600 3500 50  0001 C CNN
 F 3 "http://www.ti.com/lit/gpn/sn74LS107" H 6600 3500 50  0001 C CNN
 	2    6600 3500
@@
 F 0 "U3" H 8200 3867 50  0000 C CNN
 F 1 "74HC107" H 8200 3776 50  0000 C CNN
-F 2 "" H 8200 3500 50  0001 C CNN
+F 2 "Package_DIP:DIP-14_W7.62mm" H 8200 3500 50  0001 C CNN
 F 3 "http://www.ti.com/lit/gpn/sn74LS107" H 8200 3500 50  0001 C CNN
 	2    8200 3500
@@
 F 0 "U4" H 9800 3867 50  0000 C CNN
 F 1 "74HC107" H 9800 3776 50  0000 C CNN
-F 2 "" H 9800 3500 50  0001 C CNN
+F 2 "Package_DIP:DIP-14_W7.62mm" H 9800 3500 50  0001 C CNN
 F 3 "http://www.ti.com/lit/gpn/sn74LS107" H 9800 3500 50  0001 C CNN
 	2    9800 3500
@@
 F 0 "U5" H 11400 3867 50  0000 C CNN
 F 1 "74HC107" H 11400 3776 50  0000 C CNN
-F 2 "" H 11400 3500 50  0001 C CNN
+F 2 "Package_DIP:DIP-14_W7.62mm" H 11400 3500 50  0001 C CNN
 F 3 "http://www.ti.com/lit/gpn/sn74LS107" H 11400 3500 50  0001 C CNN
 	2    11400 3500
