File: subleq.kicad_pcb (KiCad board)
At the start: 2 copper layers, 7 parts, among them U1 74HC107, U2 74HC107, U3 74HC107, U4 74HC107, U5 74HC107, U6 74HC11, U7 74HC11

Commit message: commit after a crash, recovered backups
Parts:
- added U10: 74HC161, Package_DIP:DIP-16_W7.62mm, F.Cu at (132.1, 65.7)
- added U11: 74HC161, Package_DIP:DIP-16_W7.62mm, F.Cu at (144.8, 65.7)
- added U12: 74HC161, Package_DIP:DIP-16_W7.62mm, F.Cu at (157.5, 65.7)
- added U8: 74LS04, Package_DIP:DIP-14_W7.62mm, F.Cu at (119.4, 90.8)
- added U9: 74HC161, Package_DIP:DIP-16_W7.62mm, F.Cu at (119.4, 65.7)
- moved U2 3.81 mm to (63.5, 66.0)
- moved U3 3.81 mm to (76.2, 66.0)
- moved U4 3.81 mm to (88.9, 66.0)
- moved U6 3.81 mm to (76.2, 90.2)
- moved U7 3.81 mm to (88.9, 90.2)
- moved U1 3.81 mm to (50.8, 66.0)
- moved U5 3.81 mm to (101.6, 66.0)
Connections:
- net /~T0 renamed /CONTROL/~T0
- net /~T2 renamed /CONTROL/~T2
- net /~T3 renamed /CONTROL/~T3
- net /~T4 renamed /CONTROL/~T4
- net /~T7 renamed /CONTROL/~T7
- net /~T8 renamed /CONTROL/~T8

Commit message: calling it a night
Parts:
- added U13: 74HC257, Package_DIP:DIP-16_W7.62mm, F.Cu at (132.8, 102.5)
- added U14: 74HC257, Package_DIP:DIP-16_W7.62mm, F.Cu at (152.5, 81.6)
- added U15: 74HC257, Package_DIP:DIP-16_W7.62mm, F.Cu at (142.7, 81.6)
- added U16: 74HC257, Package_DIP:DIP-16_W7.62mm, F.Cu at (132.8, 81.6)
- added U17: AS6C1008, Package_DIP:DIP-32_W15.24mm, F.Cu at (115.4, 81.6)
- added U18: 74HC377, Package_DIP:DIP-20_W7.62mm, F.Cu at (271.7, 122.8)
- added U19: 74HC377, Package_DIP:DIP-20_W7.62mm, F.Cu at (261.8, 122.8)
- added U20: 74HC377, Package_DIP:DIP-20_W7.62mm, F.Cu at (252.0, 122.8)
- added U21: 74HC377, Package_DIP:DIP-20_W7.62mm, F.Cu at (242.1, 122.8)
- added U22: 74HC04, Package_DIP:DIP-14_W7.62mm, F.Cu at (234.5, 81.6)
- added U23: 74HC04, Package_DIP:DIP-14_W7.62mm, F.Cu at (244.3, 81.6)
- added U24: 74HC283, Package_DIP:DIP-16_W7.62mm, F.Cu at (214.8, 81.6)
- added U25: 74HC283, Package_DIP:DIP-16_W7.62mm, F.Cu at (224.6, 81.6)
- added U26: 74HC688, Package_DIP:DIP-20_W7.62mm, F.Cu at (195.1, 81.6)
- added U27: 74HC32, Package_DIP:DIP-14_W7.62mm, F.Cu at (234.5, 100.0)
- added U28: 74HC541, Package_DIP:DIP-20_W7.62mm, F.Cu at (204.9, 81.6)
- added X1: 2MHZ, Oscillator:Oscillator_DIP-8, F.Cu at (267.8, 90.4)
- U8: value 74LS04 -> 74HC04
- moved U9 116.1 mm to (217.5, 127.7)
- moved U8 114.1 mm to (227.4, 127.7)
- moved U1 102.9 mm to (115.4, 146.1)
- moved U3 99.4 mm to (135.1, 146.1)
- moved U4 87.9 mm to (125.3, 146.1)
- moved U10 83.5 mm to (188.0, 127.7)
- moved U11 81.6 mm to (197.8, 127.7)
- moved U2 80.6 mm to (115.4, 127.7)
- moved U12 79.8 mm to (207.7, 127.7)
- moved U5 75.4 mm to (145.0, 127.7)
- moved U6 69.9 mm to (135.1, 127.7)
- moved U7 52.3 mm to (125.3, 127.7)
Connections:
- net ~PC_INC renamed ~INC_PC
- U1 pad 10: ~RST -> ~ADDR_OE
- U1 pad 12: ~CLK -> CLK
- U1 pad 13: ~RST -> ~ADDR_OE
- U1 pad 9: ~CLK -> CLK
- U10 pad 1: ~RST -> ~ADDR_OE
- U10 pad 11: /PROGRAM_COUNTER/PC_Q7 -> PC_Q7
- U10 pad 12: /PROGRAM_COUNTER/PC_Q6 -> PC_Q6
- U10 pad 13: /PROGRAM_COUNTER/PC_Q5 -> PC_Q5
- U10 pad 14: /PROGRAM_COUNTER/PC_Q4 -> PC_Q4
- U10 pad 3: /PROGRAM_COUNTER/PC_D4 -> MAR_Q4
- U10 pad 4: /PROGRAM_COUNTER/PC_D5 -> MAR_Q5
- U10 pad 5: /PROGRAM_COUNTER/PC_D6 -> MAR_Q6
- U10 pad 6: /PROGRAM_COUNTER/PC_D7 -> MAR_Q7
- U10 pad 8: GND -> ~ADDR_OE
- U11 pad 1: ~RST -> ~ADDR_OE
- U11 pad 11: /PROGRAM_COUNTER/PC_Q11 -> PC_Q11
- U11 pad 12: /PROGRAM_COUNTER/PC_Q10 -> PC_Q10
- U11 pad 13: /PROGRAM_COUNTER/PC_Q9 -> PC_Q9
- U11 pad 14: /PROGRAM_COUNTER/PC_Q8 -> PC_Q8
- U11 pad 3: /PROGRAM_COUNTER/PC_D8 -> MAR_Q8
- U11 pad 4: /PROGRAM_COUNTER/PC_D9 -> MAR_Q9
- U11 pad 5: /PROGRAM_COUNTER/PC_D10 -> MAR_Q10
- U11 pad 6: /PROGRAM_COUNTER/PC_D11 -> MAR_Q11
- U11 pad 8: GND -> ~ADDR_OE
- U12 pad 1: ~RST -> ~ADDR_OE
- U12 pad 11: /PROGRAM_COUNTER/PC_Q15 -> PC_Q15
- U12 pad 12: /PROGRAM_COUNTER/PC_Q14 -> PC_Q14
- U12 pad 13: /PROGRAM_COUNTER/PC_Q13 -> PC_Q13
- U12 pad 14: /PROGRAM_COUNTER/PC_Q12 -> PC_Q12
- U12 pad 15: Net-(U12-Pad15) -> (no net)
- U12 pad 3: /PROGRAM_COUNTER/PC_D12 -> MAR_Q12
- U12 pad 4: /PROGRAM_COUNTER/PC_D13 -> MAR_Q13
- U12 pad 5: /PROGRAM_COUNTER/PC_D14 -> MAR_Q14
- U12 pad 6: /PROGRAM_COUNTER/PC_D15 -> MAR_Q15
- U12 pad 8: GND -> ~ADDR_OE
- U2 pad 10: ~RST -> ~ADDR_OE
- U2 pad 12: ~CLK -> CLK
- U2 pad 13: ~RST -> ~ADDR_OE
- U2 pad 9: ~CLK -> CLK
- U3 pad 10: ~RST -> ~ADDR_OE
- U3 pad 12: ~CLK -> CLK
- U3 pad 13: ~RST -> ~ADDR_OE
- U3 pad 9: ~CLK -> CLK
- U4 pad 10: ~RST -> ~ADDR_OE
- U4 pad 12: ~CLK -> CLK
- U4 pad 13: ~RST -> ~ADDR_OE
- U4 pad 9: ~CLK -> CLK
- U5 pad 10: ~RST -> ~ADDR_OE
- U5 pad 12: ~CLK -> CLK
- U5 pad 13: ~RST -> ~ADDR_OE
- U5 pad 9: ~CLK -> CLK
- U6 pad 8: ~ADDR_SEL -> ~SEL_ADDR_PC_MAR
- U8 pad 10: (no net) -> Net-(U25-Pad5)
- U8 pad 11: (no net) -> A4
- U8 pad 12: (no net) -> Net-(U25-Pad3)
- U8 pad 13: (no net) -> A5
- U8 pad 3: (no net) -> A1
- U8 pad 4: (no net) -> Net-(U24-Pad3)
- U8 pad 5: (no net) -> A2
- U8 pad 6: (no net) -> Net-(U24-Pad14)
- U8 pad 8: (no net) -> Net-(U17-Pad24)
- U8 pad 9: (no net) -> ~WR_MEM
- U9 pad 1: ~RST -> ~ADDR_OE
- U9 pad 11: /PROGRAM_COUNTER/PC_Q3 -> PC_Q3
- U9 pad 12: /PROGRAM_COUNTER/PC_Q2 -> PC_Q2
- U9 pad 13: /PROGRAM_COUNTER/PC_Q1 -> PC_Q1
- U9 pad 14: /PROGRAM_COUNTER/PC_Q0 -> PC_Q0
- U9 pad 3: /PROGRAM_COUNTER/PC_D0 -> MAR_Q0
- U9 pad 4: /PROGRAM_COUNTER/PC_D1 -> MAR_Q1
- U9 pad 5: /PROGRAM_COUNTER/PC_D2 -> MAR_Q2
- U9 pad 6: /PROGRAM_COUNTER/PC_D3 -> MAR_Q3
- U9 pad 8: GND -> ~ADDR_OE
